File: BLDC_Driver.kicad_sch (KiCad schematic)
At the start: 0 parts

Commit message: layout
Parts:
- added H1, H2, H3, H4: MountingHole_Pad, MountingHole:MountingHole_3.2mm_M3_Pad_Via, symbol Mechanical:MountingHole_Pad
- added J10, J6, J7, J8, J9: Conn_01x01, Connector_Wire:SolderWire-2sqmm_1x01_D2mm_OD3.9mm, symbol Connector_Generic:Conn_01x01
- added J5: CAN, Connector_PinSocket_2.54mm:PinSocket_1x03_P2.54mm_Vertical, symbol PCM_4ms_Connector:Conn_01x03
Connections:
- net Connectivity/CAN_H: now also J5.1 (Pin_1)
- net Connectivity/CAN_L: now also J5.2 (Pin_2)
- net OUT1: now also J6.1 (Pin_1)
- net OUT2: now also J9.1 (Pin_1)
- net OUT3: now also J10.1 (Pin_1)
- new net GND: H1.1, H2.1, H3.1, H4.1, J5.3 (Pin_3), J7.1 (Pin_1)
- new net VM: J8.1 (Pin_1)

Commit message: All DONE >?git add .git add .
Parts:
- removed J10, J6, J9: Conn_01x01, Connector_Wire:SolderWire-2sqmm_1x01_D2mm_OD3.9mm, symbol Connector_Generic:Conn_01x01
- added J12: Screw_Terminal_01x03, TerminalBlock_RND:TerminalBlock_RND_205-00068_1x03_P7.50mm_Horizontal, symbol Connector:Screw_Terminal_01x03
Connections:
- net OUT1: now also J12.1 (Pin_1)
- net OUT2: now also J12.2 (Pin_2)
- net OUT3: now also J12.3 (Pin_3)
Other:
- sheet Connectivity ports: added USB_DM, USB_DP; removed none
- sheet MCU ports: added USB_DM, USB_DP; removed DAC1, DAC2
- sheet Op_amp ports: added none; removed DAC1, DAC2
