File: Connectivity.kicad_sch (KiCad schematic)
At the start: 13 parts, among them J2 Conn_01x05, J3 Conn_ARM_SWD_TagConnect_TC203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, J4 USB_C_Receptacle_USB2.0_14P, U4 TCAN330G

Commit message: layout
Parts:
- J2: footprint (none) -> Connector_PinSocket_2.54mm:PinSocket_1x05_P2.54mm_Vertical
- J3, TP4, TP5: now not fitted
- J4: footprint (none) -> Connector_USB:USB_C_Receptacle_Amphenol_12401610E4-2A_CircularHoles
Changed lines of the file:
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@@
 			)
 		)
-		(property "Footprint" ""
+		(property "Footprint" "Connector_USB:USB_C_Receptacle_Amphenol_12401610E4-2A_CircularHoles"
 			(at 209.55 44.45 0)
 			(effects
@@
 		(exclude_from_sim no)
 		(in_bom no)
-		(on_board yes)
-		(dnp no)
+		(on_board no)
+		(dnp yes)
 		(fields_autoplaced yes)
 		(property "Reference" "J3"
@@
 		(in_bom yes)
 		(on_board yes)
-		(dnp no)
+		(dnp yes)
 		(fields_autoplaced yes)
 		(property "Reference" "TP5"
@@
 		(in_bom yes)
 		(on_board yes)
-		(dnp no)
+		(dnp yes)
 		(fields_autoplaced yes)
 		(property "Reference" "TP4"
@@
 			)
 		)
-		(property "Footprint" ""
+		(property "Footprint" "Connector_PinSocket_2.54mm:PinSocket_1x05_P2.54mm_Vertical"
 			(at 151.13 138.43 0)
 			(effects

Commit message: All DONE >?git add .git add .
Parts:
- removed J2: Conn_01x05, Connector_PinSocket_2.54mm:PinSocket_1x05_P2.54mm_Vertical, symbol Connector_Generic:Conn_01x05
- removed TP6, TP7: TestPoint, TestPoint:TestPoint_Pad_2.0x2.0mm, symbol Connector:TestPoint
- added J2: Conn_02x03_Counter_Clockwise, Connector_PinSocket_2.54mm:PinSocket_2x03_P2.54mm_Vertical_SMD, symbol Connector_Generic:Conn_02x03_Counter_Clockwise
- added J6: Conn_01x04, Connector_PinHeader_2.54mm:PinHeader_1x04_P2.54mm_Vertical_SMD_Pin1Left, symbol Connector_Generic:Conn_01x04
- added U2: ECMF02-2AMX6, Package_DFN_QFN:ST_UQFN-6L_1.5x1.7mm_P0.5mm, symbol Power_Protection:ECMF02-2AMX6
Connections:
- net 3V3: now also J2.6 (Pin_6), J6.1 (Pin_1)
- net GND: now also J2.4 (Pin_4), J6.4 (Pin_4), U2.3 (GND), U2.4 (NC)
- net SWCLK: now also J2.2 (Pin_2)
- net SWDIO: now also J2.1 (Pin_1)
- net SWO: now also J2.3 (Pin_3)
- net UART_RX: now also J6.2 (Pin_2)
- net UART_TX: now also J6.3 (Pin_3)
- net USB_DM: now also U2.2 (D-_in); no longer J4.A7 (D-), J4.B7 (D-)
- net USB_DP: now also U2.1 (D+_in); no longer J4.A6 (D+), J4.B6 (D+)
- net nRST: now also J2.5 (Pin_5)
- new net USB_DM_Conn: J4.A7 (D-), J4.B7 (D-), U2.5 (D-_out)
- new net USB_DP_Conn: J4.A6 (D+), J4.B6 (D+), U2.6 (D+_out)
