File: h_bridge.kicad_sch (KiCad schematic)
At the start: 21 parts, among them Q1 NMOS, Q2 NMOS, Q3 NMOS, Q4 NMOS, Q5 NMOS, Q6 NMOS

Commit message: layout
Parts:
- Q1, Q2, Q3, Q4, Q5, Q6: footprint (none) -> Package_DFN_QFN:PQFN-8-EP_6x5mm_P1.27mm_Generic
- R12, R5, R9: footprint (none) -> Resistor_SMD:R_Shunt_Vishay_WSK2512_6332Metric_T2.66mm
Changed lines of the file:
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@@
 			)
 		)
-		(property "Footprint" ""
+		(property "Footprint" "Package_DFN_QFN:PQFN-8-EP_6x5mm_P1.27mm_Generic"
 			(at 156.21 78.74 0)
 			(effects
@@
 			)
 		)
-		(property "Footprint" ""
+		(property "Footprint" "Package_DFN_QFN:PQFN-8-EP_6x5mm_P1.27mm_Generic"
 			(at 88.9 92.71 0)
 			(effects
@@
 			)
 		)
-		(property "Footprint" ""
+		(property "Footprint" "Resistor_SMD:R_Shunt_Vishay_WSK2512_6332Metric_T2.66mm"
 			(at 222.758 107.95 90)
 			(effects
@@
 			)
 		)
-		(property "Footprint" ""
+		(property "Footprint" "Package_DFN_QFN:PQFN-8-EP_6x5mm_P1.27mm_Generic"
 			(at 88.9 76.2 0)
 			(effects
@@
 			)
 		)
-		(property "Footprint" ""
+		(property "Footprint" "Resistor_SMD:R_Shunt_Vishay_WSK2512_6332Metric_T2.66mm"
 			(at 88.138 105.41 90)
 			(effects
@@
 			)
 		)
-		(property "Footprint" ""
+		(property "Footprint" "Package_DFN_QFN:PQFN-8-EP_6x5mm_P1.27mm_Generic"
 			(at 223.52 78.74 0)
 			(effects
@@
 			)
 		)
-		(property "Footprint" ""
+		(property "Footprint" "Package_DFN_QFN:PQFN-8-EP_6x5mm_P1.27mm_Generic"
 			(at 156.21 95.25 0)
 			(effects
@@
 			)
 		)
-		(property "Footprint" ""
+		(property "Footprint" "Package_DFN_QFN:PQFN-8-EP_6x5mm_P1.27mm_Generic"
 			(at 223.52 95.25 0)
 			(effects
@@
 			)
 		)
-		(property "Footprint" ""
+		(property "Footprint" "Resistor_SMD:R_Shunt_Vishay_WSK2512_6332Metric_T2.66mm"
 			(at 155.448 107.95 90)
 			(effects

Commit message: All DONE >?git add .git add .
Parts:
- removed Q1, Q2, Q3, Q4, Q5, Q6: NMOS, Package_DFN_QFN:PQFN-8-EP_6x5mm_P1.27mm_Generic, symbol Simulation_SPICE:NMOS
- added Q1, Q2, Q3, Q4, Q5, Q6: STL160N10F8, PCM_Package_SON_AKL:Infineon_PG-TDSON-8, symbol PCM_Transistor_MOSFET_AKL:STL130N8F7
Connections:
- net VSHUNT1N is gone; now on net GND: R5.3
- net VSHUNT2N is gone; now on net GND: R9.3
- net VSHUNT3N is gone; now on net GND: R12.3
- net OUT1: now also Q1.1 (S), Q1.2 (S), Q1.3 (S), Q2.5 (D)
- net OUT2: now also Q3.1 (S), Q3.2 (S), Q3.3 (S), Q4.5 (D)
- net OUT3: now also Q5.1 (S), Q5.2 (S), Q5.3 (S), Q6.5 (D)
- net VM: now also Q1.5 (D), Q3.5 (D), Q5.5 (D)
- net VSHUNT1P: now also R5.1, Q2.1 (S), Q2.2 (S), Q2.3 (S)
- net VSHUNT2P: now also R9.1, Q4.1 (S), Q4.2 (S), Q4.3 (S)
- net VSHUNT3P: now also R12.1, Q6.1 (S), Q6.2 (S), Q6.3 (S)
- net at R8.2: now also Q2.4 (G)
- net at R6.2: now also Q3.4 (G)
- net at R13.2: now also Q1.4 (G)
- net at R7.2: now also Q4.4 (G)
- net at R10.2: now also Q5.4 (G)
- net at R11.2: now also Q6.4 (G)
Other:
- moved on the sheet: R10, R11, R13, R6, R7, R8
