File: mcu.kicad_sch (KiCad schematic)
At the start: 15 parts, among them SW1 SW_Push, U1 STSPIN32G4, Y1 Crystal_GND24_Small

Commit message: layout
Parts:
- D6: footprint (none) -> Diode_SMD:D_0603_1608Metric_Pad1.05x0.95mm_HandSolder
- L1: footprint (none) -> Inductor_SMD_Wurth:L_Wurth_WE-LQSH-2512
Changed lines of the file:
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@@
 			)
 		)
-		(property "Footprint" ""
+		(property "Footprint" "Diode_SMD:D_0603_1608Metric_Pad1.05x0.95mm_HandSolder"
 			(at 26.67 156.21 0)
 			(effects
@@
 			)
 		)
-		(property "Footprint" ""
+		(property "Footprint" "Inductor_SMD_Wurth:L_Wurth_WE-LQSH-2512"
 			(at 204.47 46.99 0)
 			(effects

Commit message: All DONE >?git add .git add .
Parts:
- added J11: Conn_02x10_Counter_Clockwise, Connector_Molex:Molex_Micro-Fit_3.0_43045-2021_2x10-1MP_P3.00mm_Horizontal, symbol Connector_Generic:Conn_02x10_Counter_Clockwise
Connections:
- net 3V3: now also J11.3 (Pin_3), J11.4 (Pin_4)
- net DAC1: now also J11.15 (Pin_15)
- net DAC2: now also J11.14 (Pin_14)
- net GND: now also J11.1 (Pin_1), J11.13 (Pin_13), J11.16 (Pin_16), J11.20 (Pin_20)
- net nRST: now also J11.2 (Pin_2)
- net PC1: now reaches U1.10 (PC1)
- net PC1: now also J11.6 (Pin_6)
- net PC2: now reaches U1.11 (PC2)
- net PC2: now also J11.7 (Pin_7)
- net PC3: now reaches U1.12 (PC3)
- net PC3: now also J11.8 (Pin_8)
- net PC4: now reaches U1.21 (PC4)
- net PC4: now also J11.9 (Pin_9)
- net PB10: now reaches U1.28 (PB10)
- net PB10: now also J11.10 (Pin_10)
- net PC13: now reaches U1.3 (PC13)
- net PC15: now reaches U1.5 (PC15)
- net PA15: now reaches U1.51 (PA15)
- net PA15: now also J11.17 (Pin_17)
- net PD2: now reaches U1.53 (PD2)
- net PD2: now also J11.11 (Pin_11)
- net PB4: now reaches U1.55 (PB4)
- net PB4: now also J11.12 (Pin_12)
- net PC0: now reaches U1.9 (PC0)
- net PC0: now also J11.5 (Pin_5)
- new net CAN_H: J11.18 (Pin_18)
- new net CAN_L: J11.19 (Pin_19)
Other:
- moved on the sheet: C4, C5, C7, C8, D1, L1, R1, R2, U1, Y1
