File: power.kicad_sch (KiCad schematic)
At the start: 23 parts, among them U3 ST1S14PHR

Commit message: layout
Parts:
- C1, C2, C3: footprint Capacitor_SMD:C_0603_1608Metric_Pad1.08x0.95mm_HandSolder -> Capacitor_SMD:CP_Elec_5x4.5
- D5, D7: footprint (none) -> Diode_SMD:D_0603_1608Metric_Pad1.05x0.95mm_HandSolder
- L2: footprint (none) -> Inductor_SMD_Wurth:L_Wurth_WE-LQSH-4020
Changed lines of the file:
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@@
 			)
 		)
-		(property "Footprint" ""
+		(property "Footprint" "Diode_SMD:D_0603_1608Metric_Pad1.05x0.95mm_HandSolder"
 			(at 100.33 72.39 0)
 			(effects
@@
 			)
 		)
-		(property "Footprint" ""
+		(property "Footprint" "Inductor_SMD_Wurth:L_Wurth_WE-LQSH-4020"
 			(at 69.85 72.39 0)
 			(effects
@@
 			)
 		)
-		(property "Footprint" "Capacitor_SMD:C_0603_1608Metric_Pad1.08x0.95mm_HandSolder"
+		(property "Footprint" "Capacitor_SMD:CP_Elec_5x4.5"
 			(at 39.0652 30.48 0)
 			(effects
@@
 			)
 		)
-		(property "Footprint" ""
+		(property "Footprint" "Diode_SMD:D_0603_1608Metric_Pad1.05x0.95mm_HandSolder"
 			(at 66.04 33.02 0)
 			(effects
@@
 			)
 		)
-		(property "Footprint" "Capacitor_SMD:C_0603_1608Metric_Pad1.08x0.95mm_HandSolder"
+		(property "Footprint" "Capacitor_SMD:CP_Elec_5x4.5"
 			(at 25.0952 30.48 0)
 			(effects
@@
 			)
 		)
-		(property "Footprint" "Capacitor_SMD:C_0603_1608Metric_Pad1.08x0.95mm_HandSolder"
+		(property "Footprint" "Capacitor_SMD:CP_Elec_5x4.5"
 			(at 53.0352 30.48 0)
 			(effects

Commit message: All DONE >?git add .git add .
Parts:
- removed D7: D, Diode_SMD:D_0603_1608Metric_Pad1.05x0.95mm_HandSolder, symbol Device:D
- added C31: 100n, Capacitor_SMD:C_0603_1608Metric_Pad1.08x0.95mm_HandSolder, symbol Device:C
- added D7: ESH2PB, Diode_SMD:D_SMP_DO-220AA, symbol Diode:ESH2PB
Connections:
- net 3V3: now also C31.1
- net 5V: now also C16.1, C17.1, L2.2, R14.1, D7.1 (K)
- net GND: now also C31.2, D7.2 (A)
Other:
- moved on the sheet: C22, C23, C24, R31

Commit message: current changes as of production
Parts:
- C1, C2, C3: footprint Capacitor_SMD:CP_Elec_5x4.5 -> Capacitor_SMD:C_Elec_6.3x7.7
Changed lines of the file:
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@@
 			)
 		)
-		(property "Footprint" "Capacitor_SMD:CP_Elec_5x4.5"
+		(property "Footprint" "Capacitor_SMD:C_Elec_6.3x7.7"
 			(at 39.0652 30.48 0)
 			(effects
@@
 			)
 		)
-		(property "Footprint" "Capacitor_SMD:CP_Elec_5x4.5"
+		(property "Footprint" "Capacitor_SMD:C_Elec_6.3x7.7"
 			(at 25.0952 30.48 0)
 			(effects
@@
 			)
 		)
-		(property "Footprint" "Capacitor_SMD:CP_Elec_5x4.5"
+		(property "Footprint" "Capacitor_SMD:C_Elec_6.3x7.7"
 			(at 53.0352 30.48 0)
 			(effects
